Commit message: added lap timer environment

File: ifl_hs_track-master/src/ifl_track_gazebo/models/ifl_track.urdf (robot description, URDF)
Before this commit: robot ifl_track, 1 links, 0 joints
Links:
- added link detector; visual cylinder length=0.015 radius=0.01
- added link start_line; visual box size=0.9 0.09 0.003
Joints:
- added joint fix_box1: type fixed, parent ifl_track, child start_line, origin xyz=-4.123117 -1.463373 0.01 rpy=0 0 0
- added joint fix_detector: type fixed, parent ifl_track, child detector, origin xyz=-3.68 -1.463373 0.1 rpy=0 0 -3.14
